File: electronics/SimpleMP4.sch (KiCad schematic (older format))
At the start: 124 parts, among them J1 USB_OTG, J2 DISPLAY, Q1 8050, Q2 SI2305, Q3 SI2305, Q4 8050, Q5 8550, Q6 SI2305, Q7 8550, U1 OCP8020, U2 RK2608, U3 OCP2150TW18A, U4 OCP1240, U5 MT25QL128ABA, U6 K9HCG08U1M-PCB0/PIB0, U7 K4S641632N, U8 TRS_5PIN, U9 MMC/SD_SOCKET, Y1 24MHz

Commit message: added netlist
Parts:
- RN1: value 1K*4 -> 5R
Changed lines of the file:
@@
 LIBS:contrib
 LIBS:valves
-LIBS:SS312SAH4-R
-LIBS:SI2323CDS-T1-GE3
-LIBS:SKHLAAA010
-LIBS:ocp8020
-LIBS:ocp7190
-LIBS:sct102bc
-LIBS:sd_socket
-LIBS:ocp21050tw18a
-LIBS:cr1937
-LIBS:K9HCG08U1M
-LIBS:K4S641632N
-LIBS:RK2608
-LIBS:ocp1240
-LIBS:zled7012
-LIBS:trs_5pin
-LIBS:mt25ql128aba
+LIBS:SimpleMP4
 LIBS:SimpleMP4-cache
 EELAYER 25 0
@@
 P 14350 3050
 F 0 "RN1" V 14050 3050 50  0000 C CNN
-F 1 "1K*4" H 14400 3250 50  0000 C CNN
+F 1 "5R" H 14400 3250 50  0000 C CNN
 F 2 "Resistors_THT:R_Array_SIP5" V 14625 3050 50  0001 C CNN
 F 3 "" H 14350 3050 50  0001 C CNN

Commit message: finalizing part values
Parts:
- C25: value 30P* -> 30pF
- R16: value 390K* -> 390K
Changed lines of the file:
@@
 $EndComp
 $Comp
-L GND #PWR6
+L GND #PWR01
 U 1 1 5A2F7D9D
 P 1700 1550
-F 0 "#PWR6" H 1700 1300 50  0001 C CNN
+F 0 "#PWR01" H 1700 1300 50  0001 C CNN
 F 1 "GND" H 1700 1400 50  0000 C CNN
 F 2 "" H 1700 1550 50  0001 C CNN
@@
 $EndComp
 $Comp
-L +5V #PWR9
+L +5V #PWR02
 U 1 1 5A2F8222
 P 2150 800
-F 0 "#PWR9" H 2150 650 50  0001 C CNN
+F 0 "#PWR02" H 2150 650 50  0001 C CNN
 F 1 "+5V" H 2150 940 50  0000 C CNN
 F 2 "" H 2150 800 50  0001 C CNN
@@
 $EndComp
 $Comp
-L GND #PWR19
+L GND #PWR03
 U 1 1 5A2F909B
 P 5750 1800
-F 0 "#PWR19" H 5750 1550 50  0001 C CNN
+F 0 "#PWR03" H 5750 1550 50  0001 C CNN
 F 1 "GND" H 5750 1650 50  0000 C CNN
 F 2 "" H 5750 1800 50  0001 C CNN
@@
 $EndComp
 $Comp
-L GND #PWR24
+L GND #PWR04
 U 1 1 5A2F9CC3
 P 7300 1500
-F 0 "#PWR24" H 7300 1250 50  0001 C CNN
+F 0 "#PWR04" H 7300 1250 50  0001 C CNN
 F 1 "GND" H 7300 1350 50  0000 C CNN
 F 2 "" H 7300 1500 50  0001 C CNN
@@
 $EndComp
 $Comp
-L +5V #PWR17
+L +5V #PWR05
 U 1 1 5A2FA3D0
 P 5050 800
-F 0 "#PWR17" H 5050 650 50  0001 C CNN
+F 0 "#PWR05" H 5050 650 50  0001 C CNN
 F 1 "+5V" H 5050 940 50  0000 C CNN
 F 2 "" H 5050 800 50  0001 C CNN
@@
 $EndComp
 $Comp
-L +5V #PWR3
+L +5V #PWR06
 U 1 1 5A2FC6CF
 P 900 2300
-F 0 "#PWR3" H 900 2150 50  0001 C CNN
+F 0 "#PWR06" H 900 2150 50  0001 C CNN
 F 1 "+5V" H 900 2440 50  0000 C CNN
 F 2 "" H 900 2300 50  0001 C CNN
@@
 $EndComp
 $Comp
-L GND #PWR4
+L GND #PWR07
 U 1 1 5A2FC7FF
 P 900 2750
-F 0 "#PWR4" H 900 2500 50  0001 C CNN
+F 0 "#PWR07" H 900 2500 50  0001 C CNN
 F 1 "GND" H 900 2600 50  0000 C CNN
 F 2 "" H 900 2750 50  0001 C CNN
@@
 $EndComp
 $Comp
-L GND #PWR10
+L GND #PWR08
 U 1 1 5A2FC9DB
 P 2500 2550
-F 0 "#PWR10" H 2500 2300 50  0001 C CNN
+F 0 "#PWR08" H 2500 2300 50  0001 C CNN
 F 1 "GND" H 2500 2400 50  0000 C CNN
 F 2 "" H 2500 2550 50  0001 C CNN
@@
 $EndComp
 $Comp
-L VCC #PWR11
+L VCC #PWR09
 U 1 1 5A2FCDE3
 P 2700 2200
-F 0 "#PWR11" H 2700 2050 50  0001 C CNN
+F 0 "#PWR09" H 2700 2050 50  0001 C CNN
 F 1 "VCC" H 2700 2350 50  0000 C CNN
 F 2 "" H 2700 2200 50  0001 C CNN
@@
 $EndComp
 $Comp
-L GND #PWR30
+L GND #PWR010
 U 1 1 5A30ADED
 P 13700 7100
-F 0 "#PWR30" H 13700 6850 50  0001 C CNN
+F 0 "#PWR010" H 13700 6850 50  0001 C CNN
 F 1 "GND" H 13700 6950 50  0000 C CNN
 F 2 "" H 13700 7100 50  0001 C CNN
@@
 $EndComp
 $Comp
-L GND #PWR31
+L GND #PWR011
 U 1 1 5A30B9EE
 P 13700 8000
-F 0 "#PWR31" H 13700 7750 50  0001 C CNN
+F 0 "#PWR011" H 13700 7750 50  0001 C CNN
 F 1 "GND" H 13700 7850 50  0000 C CNN
 F 2 "" H 13700 8000 50  0001 C CNN
@@
 SD_DET
 $Comp
-L VCC #PWR32
+L VCC #PWR012
 U 1 1 5A30D7BC
 P 15500 6400
-F 0 "#PWR32" H 15500 6250 50  0001 C CNN
+F 0 "#PWR012" H 15500 6250 50  0001 C CNN
 F 1 "VCC" H 15500 6550 50  0000 C CNN
 F 2 "" H 15500 6400 50  0001 C CNN
@@
 $EndComp
 $Comp
-L GND #PWR33
+L GND #PWR013
 U 1 1 5A30E0B4
 P 15500 6900
-F 0 "#PWR33" H 15500 6650 50  0001 C CNN
+F 0 "#PWR013" H 15500 6650 50  0001 C CNN
 F 1 "GND" H 15500 6750 50  0000 C CNN
 F 2 "" H 15500 6900 50  0001 C CNN
@@
 $EndComp
 $Comp
-L GND #PWR16
+L GND #PWR014
 U 1 1 5A3110DD
 P 5000 3400
-F 0 "#PWR16" H 5000 3150 50  0001 C CNN
+F 0 "#PWR014" H 5000 3150 50  0001 C CNN
 F 1 "GND" H 5000 3250 50  0000 C CNN
 F 2 "" H 5000 3400 50  0001 C CNN
@@
 P 5900 3150
 F 0 "R16" V 5800 3200 50  0000 C CNN
-F 1 "390K*" V 5900 3150 50  0000 C CNN
+F 1 "390K" V 5900 3150 50  0000 C CNN
 F 2 "" V 5830 3150 50  0001 C CNN
 F 3 "" H 5900 3150 50  0001 C CNN
@@
 P 6100 3150
 F 0 "C25" H 6000 3050 50  0000 L CNN
-F 1 "30P*" H 5950 3250 50  0000 L CNN
+F 1 "30pF" H 5950 3250 50  0000 L CNN
 F 2 "" H 6138 3000 50  0001 C CNN
 F 3 "" H 6100 3150 50  0001 C CNN
@@
 $EndComp
 $Comp
-L GND #PWR25
+L GND #PWR015
 U 1 1 5A3132B8
 P 7550 3550
-F 0 "#PWR25" H 7550 3300 50  0001 C CNN
+F 0 "#PWR015" H 7550 3300 50  0001 C CNN
 F 1 "GND" H 7550 3400 50  0000 C CNN
 F 2 "" H 7550 3550 50  0001 C CNN
@@
 $EndComp
 $Comp
-L GND #PWR29
+L GND #PWR016
 U 1 1 5A343B54
 P 9550 10350
-F 0 "#PWR29" H 9550 10100 50  0001 C CNN
+F 0 "#PWR016" H 9550 10100 50  0001 C CNN
 F 1 "GND" H 9550 10200 50  0000 C CNN
 F 2 "" H 9550 10350 50  0001 C CNN
@@
 $EndComp
 $Comp
-L GND #PWR5
+L GND #PWR017
 U 1 1 5A339B3B
 P 1200 5800
-F 0 "#PWR5" H 1200 5550 50  0001 C CNN
+F 0 "#PWR017" H 1200 5550 50  0001 C CNN
 F 1 "GND" H 1200 5650 50  0000 C CNN
 F 2 "" H 1200 5800 50  0001 C CNN
@@
 $EndComp
 $Comp
-L GND #PWR2
+L GND #PWR018
 U 1 1 5A33B99A
 P 800 6200
-F 0 "#PWR2" H 800 5950 50  0001 C CNN
+F 0 "#PWR018" H 800 5950 50  0001 C CNN
 F 1 "GND" H 800 6050 50  0000 C CNN
 F 2 "" H 800 6200 50  0001 C CNN
@@
 $EndComp
 $Comp
-L GND #PWR1
+L GND #PWR019
 U 1 1 5A33EAE7
 P 700 7600
-F 0 "#PWR1" H 700 7350 50  0001 C CNN
+F 0 "#PWR019" H 700 7350 50  0001 C CNN
 F 1 "GND" H 700 7450 50  0000 C CNN
 F 2 "" H 700 7600 50  0001 C CNN
@@
 $EndComp
 $Comp
-L GND #PWR13
+L GND #PWR020
 U 1 1 5A34B5E9
 P 3900 10400
-F 0 "#PWR13" H 3900 10150 50  0001 C CNN
+F 0 "#PWR020" H 3900 10150 50  0001 C CNN
 F 1 "GND" H 3900 10250 50  0000 C CNN
 F 2 "" H 3900 10400 50  0001 C CNN
@@
 $EndComp
 $Comp
-L GND #PWR21
+L GND #PWR021
 U 1 1 5A354E3A
 P 6200 10700
-F 0 "#PWR21" H 6200 10450 50  0001 C CNN
+F 0 "#PWR021" H 6200 10450 50  0001 C CNN
 F 1 "GND" H 6200 10550 50  0000 C CNN
 F 2 "" H 6200 10700 50  0001 C CNN
@@
 $EndComp
 $Comp
-L GND #PWR28
+L GND #PWR022
 U 1 1 5A36AE0A
 P 8250 8850
-F 0 "#PWR28" H 8250 8600 50  0001 C CNN
+F 0 "#PWR022" H 8250 8600 50  0001 C CNN
 F 1 "GND" H 8250 8700 50  0000 C CNN
 F 2 "" H 8250 8850 50  0001 C CNN
@@
 $EndComp
 $Comp
-L GND #PWR27
+L GND #PWR023
 U 1 1 5A36EE2E
 P 7600 7800
-F 0 "#PWR27" H 7600 7550 50  0001 C CNN
+F 0 "#PWR023" H 7600 7550 50  0001 C CNN
 F 1 "GND" H 7600 7650 50  0000 C CNN
 F 2 "" H 7600 7800 50  0001 C CNN
@@
 $EndComp
 $Comp
-L GND #PWR26
+L GND #PWR024
 U 1 1 5A372A47
 P 7550 7100
-F 0 "#PWR26" H 7550 6850 50  0001 C CNN
+F 0 "#PWR024" H 7550 6850 50  0001 C CNN
 F 1 "GND" H 7550 6950 50  0000 C CNN
 F 2 "" H 7550 7100 50  0001 C CNN
@@
 $EndComp
 $Comp
-L GND #PWR23
+L GND #PWR025
 U 1 1 5A373658
 P 6750 5900
-F 0 "#PWR23" H 6750 5650 50  0001 C CNN
+F 0 "#PWR025" H 6750 5650 50  0001 C CNN
 F 1 "GND" H 6750 5750 50  0000 C CNN
 F 2 "" H 6750 5900 50  0001 C CNN
@@
 $EndComp
 $Comp
-L GND #PWR22
+L GND #PWR026
 U 1 1 5A37A4B7
 P 6750 5650
-F 0 "#PWR22" H 6750 5400 50  0001 C CNN
+F 0 "#PWR026" H 6750 5400 50  0001 C CNN
 F 1 "GND" H 6750 5500 50  0000 C CNN
 F 2 "" H 6750 5650 50  0001 C CNN
@@
 $EndComp
 $Comp
-L GND #PWR20
+L GND #PWR027
 U 1 1 5A37F849
 P 6000 4650
-F 0 "#PWR20" H 6000 4400 50  0001 C CNN
+F 0 "#PWR027" H 6000 4400 50  0001 C CNN
 F 1 "GND" H 6000 4500 50  0000 C CNN
 F 2 "" H 6000 4650 50  0001 C CNN
@@
 $EndComp
 $Comp
-L GND #PWR18
+L GND #PWR028
 U 1 1 5A380FBA
 P 5200 4350
-F 0 "#PWR18" H 5200 4100 50  0001 C CNN
+F 0 "#PWR028" H 5200 4100 50  0001 C CNN
 F 1 "GND" H 5200 4200 50  0000 C CNN
 F 2 "" H 5200 4350 50  0001 C CNN
@@
 $EndComp
 $Comp
-L GND #PWR15
+L GND #PWR029
 U 1 1 5A383D80
 P 4700 4400
-F 0 "#PWR15" H 4700 4150 50  0001 C CNN
+F 0 "#PWR029" H 4700 4150 50  0001 C CNN
 F 1 "GND" H 4700 4250 50  0000 C CNN
 F 2 "" H 4700 4400 50  0001 C CNN
@@
 $EndComp
 $Comp
-L GND #PWR14
+L GND #PWR030
 U 1 1 5A38685D
 P 4200 4400
-F 0 "#PWR14" H 4200 4150 50  0001 C CNN
+F 0 "#PWR030" H 4200 4150 50  0001 C CNN
 F 1 "GND" H 4200 4250 50  0000 C CNN
 F 2 "" H 4200 4400 50  0001 C CNN
@@
 $EndComp
 $Comp
-L GND #PWR12
+L GND #PWR031
 U 1 1 5A394DCC
 P 3050 3550
-F 0 "#PWR12" H 3050 3300 50  0001 C CNN
+F 0 "#PWR031" H 3050 3300 50  0001 C CNN
 F 1 "GND" H 3050 3400 50  0000 C CNN
 F 2 "" H 3050 3550 50  0001 C CNN
@@
 $EndComp
 $Comp
-L VCC #PWR7
+L VCC #PWR032
 U 1 1 5A39B52E
 P 1700 3450
-F 0 "#PWR7" H 1700 3300 50  0001 C CNN
+F 0 "#PWR032" H 1700 3300 50  0001 C CNN
 F 1 "VCC" H 1700 3600 50  0000 C CNN
 F 2 "" H 1700 3450 50  0001 C CNN
@@
 $EndComp
 $Comp
-L GND #PWR8
+L GND #PWR033
 U 1 1 5A39B6E0
 P 1700 4450
-F 0 "#PWR8" H 1700 4200 50  0001 C CNN
+F 0 "#PWR033" H 1700 4200 50  0001 C CNN
 F 1 "GND" H 1700 4300 50  0000 C CNN
 F 2 "" H 1700 4450 50  0001 C CNN

Commit message: updated schematics
Parts:
- C1, C10, C11, C12, C13, C14, C15, C16, C17, C18, C19, C2, C21, C22, C25, C26, C27, C28, C29, C3, C33, C34, C36, C37, C38, C39, C4, C40, C41, C42, C43, C44, C46, C47, C7, C8, C9: footprint (none) -> Capacitors_SMD:C_0603
- C20, C23, C24, C30, C31, C32, C35, C45, C5, C6: footprint (none) -> Capacitors_SMD:CP_Elec_4x4.5
- D1, D2: footprint (none) -> Diodes_SMD:D_SOD-123
- J1: footprint (none) -> Connectors:USB_Mini-B
- L1, L10, L4, L6, L7, L8, L9: footprint (none) -> Inductors_SMD:L_0603
- Q1, Q4, Q5, Q7, U4: footprint (none) -> TO_SOT_Packages_SMD:SOT-23
- Q2, Q3, Q6: footprint SOT23 -> TO_SOT_Packages_SMD:SOT-23
- R1, R17, R20, R21, R24, R25, R26, R27, R28, R29, R30, R31, R32, R33, R34, R35, R36, R5, R7, R8, R9: footprint (none) -> Resistors_SMD:R_0603
- R10, R11, R12, R13, R14, R15, R16, R18, R19, R2, R22, R23, R3, R4, R6: footprint (none) -> Resistors_SMD:R_0805
- U1, U3: footprint (none) -> TO_SOT_Packages_SMD:SOT-23-5
- U2: footprint MODULE -> Housings_QFP:LQFP-128_14x14mm_Pitch0.4mm
- U6: footprint MODULE -> Housings_SSOP:TSOP-I-48_18.4x12mm_Pitch0.5mm
- U8: footprint (none) -> Connectors:Stereo_Jack_3.5mm_Switch_Ledino_KB3SPRS
- U9: footprint (none) -> Connectors:SD_Card_Receptacle

Commit message: placed most components around rk2608
Parts:
- B1, B3, B4, B5, B6: footprint SKHLAAA010 -> SKHLAAA010:SKHLAAA010
- BT1: footprint (none) -> Connectors_JST:JST_PH_B2B-PH-SM4-TB_02x2.00mm_Straight
- S1: footprint SW_SS312SAH4-R -> SS312SAH4-R:SW_SS312SAH4-R
- U5: footprint (none) -> SOP-8:SOP-8
- U7: footprint MODULE -> TSOP-54:TSOP-54
- Y1: footprint (none) -> Crystals:Crystal_SMD_HC49-SD
Changed lines of the file:
@@
 F 0 "BT1" H 5750 1600 50  0000 L CNN
 F 1 "LI-3.6V" H 5450 1600 50  0000 L CNN
-F 2 "" V 5750 1710 50  0001 C CNN
+F 2 "Connectors_JST:JST_PH_B2B-PH-SM4-TB_02x2.00mm_Straight" V 5750 1710 50  0001 C CNN
 F 3 "" V 5750 1710 50  0001 C CNN
 	1    5750 1650
@@
 F 0 "S1" H 5150 1510 50  0000 L BNN
 F 1 "ON/OFF" H 5200 1000 50  0000 L BNN
-F 2 "SW_SS312SAH4-R" H 5350 1300 50  0001 L BNN
+F 2 "SS312SAH4-R:SW_SS312SAH4-R" H 5350 1300 50  0001 L BNN
 F 3 "NKK Switches" H 5350 1300 50  0001 L BNN
 F 4 "Good" H 5350 1300 50  0001 L BNN "Availability"
@@
 F 0 "B1" H 5900 1800 50  0000 L BNN
 F 1 "PLAY/STOP" H 5850 1600 50  0000 L BNN
-F 2 "SKHLAAA010" H 6000 1700 50  0001 L BNN
+F 2 "SKHLAAA010:SKHLAAA010" H 6000 1700 50  0001 L BNN
 F 3 "SKHLAAA010" H 6000 1700 50  0001 L BNN
 F 4 "None" H 6000 1700 50  0001 L BNN "Package"
@@
 F 0 "U7" H 10400 8550 50  0000 C CNN
 F 1 "K4S641632N" H 10400 10200 50  0000 C CNN
-F 2 "MODULE" H 10400 8650 50  0001 C CNN
+F 2 "TSOP-54:TSOP-54" H 10400 8650 50  0001 C CNN
 F 3 "DOCUMENTATION" H 10400 8650 50  0001 C CNN
 	1    10400 8650
@@
 F 0 "B3" H 5900 10250 50  0000 L BNN
 F 1 "VOL" H 6350 10200 50  0000 L BNN
-F 2 "SKHLAAA010" H 6050 10200 50  0001 L BNN
+F 2 "SKHLAAA010:SKHLAAA010" H 6050 10200 50  0001 L BNN
 F 3 "SKHLAAA010" H 6050 10200 50  0001 L BNN
 F 4 "None" H 6050 10200 50  0001 L BNN "Package"
@@
 F 0 "B4" H 5900 10400 50  0000 L BNN
 F 1 "FFD/>>" H 6350 10350 50  0000 L BNN
-F 2 "SKHLAAA010" H 6050 10350 50  0001 L BNN
+F 2 "SKHLAAA010:SKHLAAA010" H 6050 10350 50  0001 L BNN
 F 3 "SKHLAAA010" H 6050 10350 50  0001 L BNN
 F 4 "None" H 6050 10350 50  0001 L BNN "Package"
@@
 F 0 "B5" H 5900 10550 50  0000 L BNN
 F 1 "FFW/<<" H 6350 10500 50  0000 L BNN
-F 2 "SKHLAAA010" H 6050 10500 50  0001 L BNN
+F 2 "SKHLAAA010:SKHLAAA010" H 6050 10500 50  0001 L BNN
 F 3 "SKHLAAA010" H 6050 10500 50  0001 L BNN
 F 4 "None" H 6050 10500 50  0001 L BNN "Package"
@@
 F 0 "B6" H 5900 10700 50  0000 L BNN
 F 1 "MENU" H 6350 10650 50  0000 L BNN
-F 2 "SKHLAAA010" H 6050 10650 50  0001 L BNN
+F 2 "SKHLAAA010:SKHLAAA010" H 6050 10650 50  0001 L BNN
 F 3 "SKHLAAA010" H 6050 10650 50  0001 L BNN
 F 4 "None" H 6050 10650 50  0001 L BNN "Package"
@@
 F 0 "Y1" H 3050 4100 50  0000 C CNN
 F 1 "24MHz" H 3050 3800 50  0000 C CNN
-F 2 "" H 3050 3950 50  0001 C CNN
+F 2 "Crystals:Crystal_SMD_HC49-SD" H 3050 3950 50  0001 C CNN
 F 3 "" H 3050 3950 50  0001 C CNN
 	1    3050 3950
@@
 F 0 "U5" H 10350 3400 60  0000 C CNN
 F 1 "MT25QL128ABA" H 10350 3900 60  0000 C CNN
-F 2 "" H 10300 3050 60  0001 C CNN
+F 2 "SOP-8:SOP-8" H 10300 3050 60  0001 C CNN
 F 3 "" H 10300 3050 60  0001 C CNN
 	1    10300 3450

Commit message: fixed minor error in schematic'
Connections:
- net GND: now also R18.2, R23.1, R26.1
Changed lines of the file:
@@
 	13250 2500 13250 2850
 Connection ~ 13250 2850
+$Comp
+L GND #PWR?
+U 1 1 5A3F0F6A
+P 6700 2250
+F 0 "#PWR?" H 6700 2000 50  0001 C CNN
+F 1 "GND" H 6700 2100 50  0000 C CNN
+F 2 "" H 6700 2250 50  0001 C CNN
+F 3 "" H 6700 2250 50  0001 C CNN
+	1    6700 2250
+	1    0    0    -1
+$EndComp
+Wire Wire Line
+	6700 2200 6700 2250
+Connection ~ 6700 2200
 $EndSCHEMATC

Commit message: added display connector
Parts:
- B2: footprint SKHLAAA010 -> SKHLAAA010:SKHLAAA010
Changed lines of the file:
@@
 F 0 "B2" H 5900 10100 50  0000 L BNN
 F 1 "EQ" H 6350 10050 50  0000 L BNN
-F 2 "SKHLAAA010" H 6050 10050 50  0001 L BNN
+F 2 "SKHLAAA010:SKHLAAA010" H 6050 10050 50  0001 L BNN
 F 3 "SKHLAAA010" H 6050 10050 50  0001 L BNN
 F 4 "None" H 6050 10050 50  0001 L BNN "Package"
@@
 Connection ~ 13250 2850
 $Comp
-L GND #PWR?
+L GND #PWR034
 U 1 1 5A3F0F6A
 P 6700 2250
-F 0 "#PWR?" H 6700 2000 50  0001 C CNN
+F 0 "#PWR034" H 6700 2000 50  0001 C CNN
 F 1 "GND" H 6700 2100 50  0000 C CNN
 F 2 "" H 6700 2250 50  0001 C CNN

Commit message: placed more components and defined board edge
Parts:
- J2: footprint (none) -> footprints:KD024B
- L2: footprint (none) -> footprints:CR43NP-4R7MC
- R10, R11, R12, R13, R14, R15, R16, R18, R19, R2, R22, R23, R3, R4, R6: footprint Resistors_SMD:R_0805 -> Resistors_SMD:R_0603
Changed lines of the file:
@@
 F 0 "R4" V 1580 1350 50  0000 C CNN
 F 1 "1M" V 1500 1350 50  0000 C CNN
-F 2 "Resistors_SMD:R_0805" V 1430 1350 50  0001 C CNN
+F 2 "Resistors_SMD:R_0603" V 1430 1350 50  0001 C CNN
 F 3 "" H 1500 1350 50  0001 C CNN
 	1    1500 1350
@@
 F 0 "R6" V 1780 1250 50  0000 C CNN
 F 1 "1M" V 1700 1250 50  0000 C CNN
-F 2 "Resistors_SMD:R_0805" V 1630 1250 50  0001 C CNN
+F 2 "Resistors_SMD:R_0603" V 1630 1250 50  0001 C CNN
 F 3 "" H 1700 1250 50  0001 C CNN
 	1    1700 1250
@@
 F 0 "R19" V 6280 1350 50  0000 C CNN
 F 1 "100K" V 6200 1350 50  0000 C CNN
-F 2 "Resistors_SMD:R_0805" V 6130 1350 50  0001 C CNN
+F 2 "Resistors_SMD:R_0603" V 6130 1350 50  0001 C CNN
 F 3 "" H 6200 1350 50  0001 C CNN
 	1    6200 1350
@@
 F 0 "R18" V 6080 2050 50  0000 C CNN
 F 1 "100K" V 6000 2050 50  0000 C CNN
-F 2 "Resistors_SMD:R_0805" V 5930 2050 50  0001 C CNN
+F 2 "Resistors_SMD:R_0603" V 5930 2050 50  0001 C CNN
 F 3 "" H 6000 2050 50  0001 C CNN
 	1    6000 2050
@@
 F 0 "R23" V 7130 2050 50  0000 C CNN
 F 1 "100K" V 7050 2050 50  0000 C CNN
-F 2 "Resistors_SMD:R_0805" V 6980 2050 50  0001 C CNN
+F 2 "Resistors_SMD:R_0603" V 6980 2050 50  0001 C CNN
 F 3 "" H 7050 2050 50  0001 C CNN
 	1    7050 2050
@@
 F 0 "R10" V 2780 2350 50  0000 C CNN
 F 1 "100K" V 2700 2350 50  0000 C CNN
-F 2 "Resistors_SMD:R_0805" V 2630 2350 50  0001 C CNN
+F 2 "Resistors_SMD:R_0603" V 2630 2350 50  0001 C CNN
 F 3 "" H 2700 2350 50  0001 C CNN
 	1    2700 2350
@@
 F 0 "R14" V 5500 3450 50  0000 C CNN
 F 1 "150K*" V 5600 3400 50  0000 C CNN
-F 2 "Resistors_SMD:R_0805" V 5530 3400 50  0001 C CNN
+F 2 "Resistors_SMD:R_0603" V 5530 3400 50  0001 C CNN
 F 3 "" H 5600 3400 50  0001 C CNN
 	1    5600 3400
@@
 F 0 "L2" V 7250 3100 50  0000 C CNN
 F 1 "4.7uH" V 7375 3100 50  0000 C CNN
-F 2 "" H 7300 3100 50  0001 C CNN
+F 2 "footprints:CR43NP-4R7MC" H 7300 3100 50  0001 C CNN
 F 3 "" H 7300 3100 50  0001 C CNN
 	1    7300 3100
@@
 F 0 "R16" V 5800 3200 50  0000 C CNN
 F 1 "390K" V 5900 3150 50  0000 C CNN
-F 2 "Resistors_SMD:R_0805" V 5830 3150 50  0001 C CNN
+F 2 "Resistors_SMD:R_0603" V 5830 3150 50  0001 C CNN
 F 3 "" H 5900 3150 50  0001 C CNN
 	1    5900 3150
@@
 F 0 "R22" V 6900 10700 50  0000 C CNN
 F 1 "100K" V 7000 10650 50  0000 C CNN
-F 2 "Resistors_SMD:R_0805" V 6930 10650 50  0001 C CNN
+F 2 "Resistors_SMD:R_0603" V 6930 10650 50  0001 C CNN
 F 3 "" H 7000 10650 50  0001 C CNN
 	1    7000 10650
@@
 F 0 "R12" V 5100 4700 50  0000 C CNN
 F 1 "100K" V 5200 4650 50  0000 C CNN
-F 2 "Resistors_SMD:R_0805" V 5130 4650 50  0001 C CNN
+F 2 "Resistors_SMD:R_0603" V 5130 4650 50  0001 C CNN
 F 3 "" H 5200 4650 50  0001 C CNN
 	1    5200 4650
@@
 F 0 "R13" V 5300 4450 50  0000 C CNN
 F 1 "100K" V 5400 4400 50  0000 C CNN
-F 2 "Resistors_SMD:R_0805" V 5330 4400 50  0001 C CNN
+F 2 "Resistors_SMD:R_0603" V 5330 4400 50  0001 C CNN
 F 3 "" H 5400 4400 50  0001 C CNN
 	1    5400 4400
@@
 F 0 "R15" V 5550 4300 50  0000 C CNN
 F 1 "100K" V 5650 4250 50  0000 C CNN
-F 2 "Resistors_SMD:R_0805" V 5580 4250 50  0001 C CNN
+F 2 "Resistors_SMD:R_0603" V 5580 4250 50  0001 C CNN
 F 3 "" H 5650 4250 50  0001 C CNN
 	1    5650 4250
@@
 F 0 "R11" V 2950 4350 50  0000 C CNN
 F 1 "1M" V 3050 4300 50  0000 C CNN
-F 2 "Resistors_SMD:R_0805" V 2980 4300 50  0001 C CNN
+F 2 "Resistors_SMD:R_0603" V 2980 4300 50  0001 C CNN
 F 3 "" H 3050 4300 50  0001 C CNN
 	1    3050 4300
@@
 F 0 "R2" V 1200 3700 50  0000 C CNN
 F 1 "220K" V 1300 3650 50  0000 C CNN
-F 2 "Resistors_SMD:R_0805" V 1230 3650 50  0001 C CNN
+F 2 "Resistors_SMD:R_0603" V 1230 3650 50  0001 C CNN
 F 3 "" H 1300 3650 50  0001 C CNN
 	1    1300 3650
@@
 F 0 "R3" V 1350 4450 50  0000 C CNN
 F 1 "1M" V 1450 4400 50  0000 C CNN
-F 2 "Resistors_SMD:R_0805" V 1380 4400 50  0001 C CNN
+F 2 "Resistors_SMD:R_0603" V 1380 4400 50  0001 C CNN
 F 3 "" H 1450 4400 50  0001 C CNN
 	1    1450 4400
@@
 F 0 "J2" H 14850 5050 50  0000 C CNN
 F 1 "DISPLAY" V 14950 3150 50  0000 C CNN
-F 2 "" H 14850 3150 50  0001 C CNN
+F 2 "footprints:KD024B" H 14850 3150 50  0001 C CNN
 F 3 "" H 14850 3150 50  0001 C CNN
 	1    14850 3150

Commit message: pausing for now
Parts:
- U5: footprint SOP-8:SOP-8 -> footprints:SOP-8
Changed lines of the file:
@@
 F 0 "U5" H 10350 3400 60  0000 C CNN
 F 1 "MT25QL128ABA" H 10350 3900 60  0000 C CNN
-F 2 "SOP-8:SOP-8" H 10300 3050 60  0001 C CNN
+F 2 "footprints:SOP-8" H 10300 3050 60  0001 C CNN
 F 3 "" H 10300 3050 60  0001 C CNN
 	1    10300 3450
