File: electronics/SimpleMP4.sch (KiCad schematic (older format))
At the start: 130 parts, among them J1 USB_OTG, J2 DISPLAY, Q1 8050, Q2 SI2305, Q3 SI2305, Q4 8050, Q5 8550, Q6 SI2305, Q7 8550, U1 OCP8020, U2 RK2608, U3 OCP2150TW18A, U4 OCP1240, U5 MT25QL128ABA, U6 K9HCG08U1M-PCB0/PIB0, U7 K4S641632N, U8 TRS_5PIN, U9 MMC/SD_SOCKET, Y1 24MHz

Commit message: labelling components with digikey part number
Parts:
- C1, C11: value 105 -> 1uF; Digikey (none) -> 399-3118-1-ND
- C10, C12, C21, C8, C9: value 104 -> 0.1uF; Digikey (none) -> 399-1095-1-ND
- C13, C14: value 8P -> 8pF; Digikey (none) -> 1276-1817-1-ND
- C20: Digikey (none) -> PCE3857CT-ND
- C22: value 103 -> 10nF; Digikey (none) -> 478-1227-1-ND
- C25: Digikey (none) -> 1276-1021-1-ND
- D1: Digikeyy (none) -> 1N5819HW-FDICT-ND
- D2: Digikey (none) -> 1N4148W-FDIDKR-ND
- J1: value USB_OTG -> CONN USB MICRO B; Digikey (none) -> 609-4613-2-ND
- L1: Digikey (none) -> 490-14398-2-ND
- Q1, Q4: Digikey (none) -> MMSS8050-H-TPMSCT-ND
- R10, R18, R19, R23: Digikey (none) -> RR08P100KDCT-ND
- R11, R3, R4, R6: Digikey (none) -> A119955TR-ND
- R17, R26, R7, R8: Digikey (none) -> 311-10KDCT-ND
- R2: Digikey (none) -> RR08P220KDCT-ND
- R21, R24: Digikey (none) -> P47KDBCT-ND
- R9: Digikey (none) -> P12KDBCT-ND
- Y1: Digikey (none) -> 535-10233-1-ND
Changed lines of the file:
@@
 P 1050 1100
 F 0 "J1" H 850 1550 50  0000 L CNN
-F 1 "USB_OTG" H 850 1450 50  0000 L CNN
+F 1 "CONN USB MICRO B" H 850 1450 50  0000 L CNN
 F 2 "footprints:USB_Mini-B" H 1200 1050 50  0001 C CNN
 F 3 "" H 1200 1050 50  0001 C CNN
+F 4 "609-4613-2-ND" H 1050 1100 60  0001 C CNN "Digikey"
 	1    1050 1100
 	1    0    0    -1
@@
 F 2 "footprints:L_0603" H 1600 900 50  0001 C CNN
 F 3 "" H 1600 900 50  0001 C CNN
+F 4 "490-14398-2-ND" V 1600 900 60  0001 C CNN "Digikey"
 	1    1600 900
 	0    1    1    0
@@
 F 2 "footprints:R_0603" V 1430 1350 50  0001 C CNN
 F 3 "" H 1500 1350 50  0001 C CNN
+F 4 "A119955TR-ND" V 1500 1350 60  0001 C CNN "Digikey"
 	1    1500 1350
 	1    0    0    -1
@@
 F 2 "footprints:R_0603" V 1630 1250 50  0001 C CNN
 F 3 "" H 1700 1250 50  0001 C CNN
+F 4 "A119955TR-ND" V 1700 1250 60  0001 C CNN "Digikey"
 	1    1700 1250
 	1    0    0    -1
@@
 P 1950 1250
 F 0 "C9" H 1975 1350 50  0000 L CNN
-F 1 "104" H 1950 1150 50  0000 L CNN
+F 1 "0.1uF" H 1850 1150 50  0000 L CNN
 F 2 "footprints:C_0603" H 1988 1100 50  0001 C CNN
 F 3 "" H 1950 1250 50  0001 C CNN
+F 4 "399-1095-1-ND" H 1950 1250 60  0001 C CNN "Digikey"
 	1    1950 1250
 	1    0    0    -1
@@
 F 2 "footprints:R_0603" V 2080 1000 50  0001 C CNN
 F 3 "" H 2150 1000 50  0001 C CNN
+F 4 "311-10KDCT-ND" V 2150 1000 60  0001 C CNN "Digikey"
 	1    2150 1000
 	1    0    0    -1
@@
 F 2 "footprints:R_0603" V 2080 1350 50  0001 C CNN
 F 3 "" H 2150 1350 50  0001 C CNN
+F 4 "P12KDBCT-ND" V 2150 1350 60  0001 C CNN "Digikey"
 	1    2150 1350
 	1    0    0    -1
@@
 P 2400 1350
 F 0 "C12" H 2425 1450 50  0000 L CNN
-F 1 "104" H 2425 1250 50  0000 L CNN
+F 1 "0.1uF" H 2400 1250 50  0000 L CNN
 F 2 "footprints:C_0603" H 2438 1200 50  0001 C CNN
 F 3 "" H 2400 1350 50  0001 C CNN
+F 4 "399-1095-1-ND" H 2400 1350 60  0001 C CNN "Digikey"
 	1    2400 1350
 	1    0    0    -1
@@
 F 2 "footprints:R_0603" V 5930 1350 50  0001 C CNN
 F 3 "" H 6000 1350 50  0001 C CNN
+F 4 "311-10KDCT-ND" V 6000 1350 60  0001 C CNN "Digikey"
 	1    6000 1350
 	1    0    0    -1
@@
 F 2 "footprints:R_0603" V 6130 1350 50  0001 C CNN
 F 3 "" H 6200 1350 50  0001 C CNN
+F 4 "RR08P100KDCT-ND" V 6200 1350 60  0001 C CNN "Digikey"
 	1    6200 1350
 	1    0    0    -1
@@
 F 2 "footprints:R_0603" V 5930 2050 50  0001 C CNN
 F 3 "" H 6000 2050 50  0001 C CNN
+F 4 "RR08P100KDCT-ND" V 6000 2050 60  0001 C CNN "Digikey"
 	1    6000 2050
 	1    0    0    -1
@@
 F 2 "footprints:D_SOD-123" H 6250 1850 50  0001 C CNN
 F 3 "" H 6250 1850 50  0001 C CNN
+F 4 "1N4148W-FDIDKR-ND" H 6250 1850 60  0001 C CNN "Digikey"
 	1    6250 1850
 	-1   0    0    1
@@
 F 2 "footprints:R_0603" V 6780 1850 50  0001 C CNN
 F 3 "" H 6850 1850 50  0001 C CNN
+F 4 "P47KDBCT-ND" V 6850 1850 60  0001 C CNN "Digikey"
 	1    6850 1850
 	0    1    1    0
@@
 F 2 "footprints:SOT-23" H 7250 1700 50  0001 C CNN
 F 3 "" H 7050 1600 50  0001 C CNN
+F 4 "MMSS8050-H-TPMSCT-ND" V 7050 1600 60  0001 C CNN "Digikey"
 	1    7050 1600
 	0    -1   -1   0
@@
 F 2 "footprints:R_0603" V 7180 1850 50  0001 C CNN
 F 3 "" H 7250 1850 50  0001 C CNN
+F 4 "P47KDBCT-ND" V 7250 1850 60  0001 C CNN "Digikey"
 	1    7250 1850
 	0    1    1    0
@@
 F 2 "footprints:R_0603" V 6980 2050 50  0001 C CNN
 F 3 "" H 7050 2050 50  0001 C CNN
+F 4 "RR08P100KDCT-ND" V 7050 2050 60  0001 C CNN "Digikey"
 	1    7050 2050
 	-1   0    0    1
@@
 F 2 "footprints:R_0603" V 7380 2050 50  0001 C CNN
 F 3 "" H 7450 2050 50  0001 C CNN
+F 4 "311-10KDCT-ND" V 7450 2050 60  0001 C CNN "Digikey"
 	1    7450 2050
 	-1   0    0    1
@@
 F 2 "footprints:D_SOD-123" H 5350 800 50  0001 C CNN
 F 3 "" H 5350 800 50  0001 C CNN
+F 4 "1N5819HW-FDICT-ND" H 5350 800 60  0001 C CNN "Digikeyy"
 	1    5350 800
 	-1   0    0    1
@@
 P 900 2550
 F 0 "C1" H 800 2650 50  0000 L CNN
-F 1 "105" H 800 2450 50  0000 L CNN
+F 1 "1uF" H 800 2450 50  0000 L CNN
 F 2 "footprints:C_0603" H 938 2400 50  0001 C CNN
 F 3 "" H 900 2550 50  0001 C CNN
+F 4 "399-3118-1-ND" H 900 2550 60  0001 C CNN "Digikey"
 	1    900  2550
 	1    0    0    -1
@@
 P 2350 2400
 F 0 "C11" H 2375 2500 50  0000 L CNN
-F 1 "105" H 2350 2300 50  0000 L CNN
+F 1 "1uF" H 2350 2300 50  0000 L CNN
 F 2 "footprints:C_0603" H 2388 2250 50  0001 C CNN
 F 3 "" H 2350 2400 50  0001 C CNN
+F 4 "399-3118-1-ND" H 2350 2400 60  0001 C CNN "Digikey"
 	1    2350 2400
 	1    0    0    -1
@@
 F 2 "footprints:R_0603" V 2630 2350 50  0001 C CNN
 F 3 "" H 2700 2350 50  0001 C CNN
+F 4 "RR08P100KDCT-ND" V 2700 2350 60  0001 C CNN "Digikey"
 	1    2700 2350
 	-1   0    0    1
@@
 P 5000 3150
 F 0 "C20" H 5000 3250 50  0000 L CNN
-F 1 "22uF" H 5025 3050 50  0000 L CNN
+F 1 "22uF" H 4800 3050 50  0000 L CNN
 F 2 "footprints:CP_Elec_4x4.5" H 5038 3000 50  0001 C CNN
 F 3 "" H 5000 3150 50  0001 C CNN
+F 4 "PCE3857CT-ND" H 5000 3150 60  0001 C CNN "Digikey"
 	1    5000 3150
 	1    0    0    -1
@@
 P 5250 3150
 F 0 "C21" H 5150 3050 50  0000 L CNN
-F 1 "104" H 5100 3250 50  0000 L CNN
+F 1 "0.1uF" H 5100 3250 50  0000 L CNN
 F 2 "footprints:C_0603" H 5288 3000 50  0001 C CNN
 F 3 "" H 5250 3150 50  0001 C CNN
+F 4 "399-1095-1-ND" H 5250 3150 60  0001 C CNN "Digikey"
 	1    5250 3150
 	-1   0    0    1
@@
 P 5500 3150
 F 0 "C22" H 5400 3050 50  0000 L CNN
-F 1 "103" H 5350 3250 50  0000 L CNN
+F 1 "10nF" H 5350 3250 50  0000 L CNN
 F 2 "footprints:C_0603" H 5538 3000 50  0001 C CNN
 F 3 "" H 5500 3150 50  0001 C CNN
+F 4 "478-1227-1-ND" H 5500 3150 60  0001 C CNN "Digikey"
 	1    5500 3150
 	-1   0    0    1
@@
 F 2 "footprints:C_0603" H 6138 3000 50  0001 C CNN
 F 3 "" H 6100 3150 50  0001 C CNN
+F 4 "1276-1021-1-ND" H 6100 3150 60  0001 C CNN "Digikey"
 	1    6100 3150
 	-1   0    0    1
@@
 F 2 "footprints:Crystal_SMD_HC49-SD" H 3050 3950 50  0001 C CNN
 F 3 "" H 3050 3950 50  0001 C CNN
+F 4 "535-10233-1-ND" H 3050 3950 60  0001 C CNN "Digikey"
 	1    3050 3950
 	1    0    0    -1
@@
 P 2750 3800
 F 0 "C13" H 2650 3900 50  0000 L CNN
-F 1 "8P" H 2600 3700 50  0000 L CNN
+F 1 "8pF" H 2600 3700 50  0000 L CNN
 F 2 "footprints:C_0603" H 2788 3650 50  0001 C CNN
 F 3 "" H 2750 3800 50  0001 C CNN
+F 4 "1276-1817-1-ND" H 2750 3800 60  0001 C CNN "Digikey"
 	1    2750 3800
 	-1   0    0    1
@@
 P 3350 3800
 F 0 "C14" H 3250 3900 50  0000 L CNN
-F 1 "8P" H 3200 3700 50  0000 L CNN
+F 1 "8pF" H 3200 3700 50  0000 L CNN
 F 2 "footprints:C_0603" H 3388 3650 50  0001 C CNN
 F 3 "" H 3350 3800 50  0001 C CNN
+F 4 "1276-1817-1-ND" H 3350 3800 60  0001 C CNN "Digikey"
 	1    3350 3800
 	-1   0    0    1
@@
 F 2 "footprints:R_0603" V 2980 4300 50  0001 C CNN
 F 3 "" H 3050 4300 50  0001 C CNN
+F 4 "A119955TR-ND" V 3050 4300 60  0001 C CNN "Digikey"
 	1    3050 4300
 	0    1    1    0
@@
 F 2 "footprints:SOT-23" H 1800 4150 50  0001 C CNN
 F 3 "" H 1600 4050 50  0001 C CNN
+F 4 "MMSS8050-H-TPMSCT-ND" V 1600 4050 60  0001 C CNN "Digikey"
 	1    1600 4050
 	1    0    0    -1
@@
 P 1950 4050
 F 0 "C10" H 1850 4150 50  0000 L CNN
-F 1 "104" H 1800 3950 50  0000 L CNN
+F 1 "0.1uF" H 1800 3950 50  0000 L CNN
 F 2 "footprints:C_0603" H 1988 3900 50  0001 C CNN
 F 3 "" H 1950 4050 50  0001 C CNN
+F 4 "399-1095-1-ND" H 1950 4050 60  0001 C CNN "Digikey"
 	1    1950 4050
 	-1   0    0    1
@@
 F 2 "footprints:R_0603" V 1630 3650 50  0001 C CNN
 F 3 "" H 1700 3650 50  0001 C CNN
+F 4 "311-10KDCT-ND" V 1700 3650 60  0001 C CNN "Digikey"
 	1    1700 3650
 	-1   0    0    1
@@
 F 2 "footprints:R_0603" V 1230 3650 50  0001 C CNN
 F 3 "" H 1300 3650 50  0001 C CNN
+F 4 "RR08P220KDCT-ND" V 1300 3650 60  0001 C CNN "Digikey"
 	1    1300 3650
 	-1   0    0    1
@@
 F 2 "footprints:R_0603" V 1380 4400 50  0001 C CNN
 F 3 "" H 1450 4400 50  0001 C CNN
+F 4 "A119955TR-ND" V 1450 4400 60  0001 C CNN "Digikey"
 	1    1450 4400
 	0    -1   -1   0
@@
 P 1500 3500
 F 0 "C8" V 1550 3550 50  0000 L CNN
-F 1 "104" H 1350 3400 50  0000 L CNN
+F 1 "0.1uF" H 1350 3400 50  0000 L CNN
 F 2 "footprints:C_0603" H 1538 3350 50  0001 C CNN
 F 3 "" H 1500 3500 50  0001 C CNN
+F 4 "399-1095-1-ND" V 1500 3500 60  0001 C CNN "Digikey"
 	1    1500 3500
 	0    -1   -1   0

Commit message: SimpleMP4
Parts:
- C31, C45: Digikey (none) -> PCE3878CT-ND
- C33: value 103 -> 10nF; Digikey (none) -> 478-1227-1-ND
- C39, C40: value 473 -> 47nF; Digikey (none) -> 399-9096-1-ND
- C43, C44, C46: Digikey (none) -> 399-1095-1-ND
- L10, L4, L6, L7, L8, L9: Digikey (none) -> 490-14398-2-ND
- L2: Digikey (none) -> 308-1527-1-ND
- R14: Digikey (none) -> P150KDBCT-ND
- R16: Digikey (none) -> A119962CT-ND
- R27, R28: Digikey (none) -> A103049TR-ND
- R29, R30, R31, R32, R33, R34: Digikey (none) -> P47KDBCT-ND
- R35, R36: Digikey (none) -> 311-10KDCT-ND
- R37, R38, R39, R40: Digikey (none) -> MCT0603-33.0-CFCT-ND
Changed lines of the file:
@@
 F 2 "footprints:R_0603" V 13680 6650 50  0001 C CNN
 F 3 "" H 13750 6650 50  0001 C CNN
+F 4 "P47KDBCT-ND" V 13750 6650 60  0001 C CNN "Digikey"
 	1    13750 6650
 	1    0    0    -1
@@
 F 2 "footprints:R_0603" V 13930 6650 50  0001 C CNN
 F 3 "" H 14000 6650 50  0001 C CNN
+F 4 "P47KDBCT-ND" V 14000 6650 60  0001 C CNN "Digikey"
 	1    14000 6650
 	1    0    0    -1
@@
 F 2 "footprints:R_0603" V 14180 6650 50  0001 C CNN
 F 3 "" H 14250 6650 50  0001 C CNN
+F 4 "P47KDBCT-ND" V 14250 6650 60  0001 C CNN "Digikey"
 	1    14250 6650
 	1    0    0    -1
@@
 F 2 "footprints:R_0603" V 14430 6650 50  0001 C CNN
 F 3 "" H 14500 6650 50  0001 C CNN
+F 4 "P47KDBCT-ND" V 14500 6650 60  0001 C CNN "Digikey"
 	1    14500 6650
 	1    0    0    -1
@@
 F 2 "footprints:R_0603" V 14680 6650 50  0001 C CNN
 F 3 "" H 14750 6650 50  0001 C CNN
+F 4 "P47KDBCT-ND" V 14750 6650 60  0001 C CNN "Digikey"
 	1    14750 6650
 	1    0    0    -1
@@
 F 2 "footprints:R_0603" V 14930 6650 50  0001 C CNN
 F 3 "" H 15000 6650 50  0001 C CNN
+F 4 "P47KDBCT-ND" V 15000 6650 60  0001 C CNN "Digikey"
 	1    15000 6650
 	1    0    0    -1
@@
 F 2 "footprints:CP_Elec_4x4.5" H 15538 6550 50  0001 C CNN
 F 3 "" H 15500 6700 50  0001 C CNN
+F 4 "PCE3878CT-ND" H 15500 6700 60  0001 C CNN "Digikey"
 	1    15500 6700
 	1    0    0    -1
@@
 F 2 "footprints:R_0603" V 5530 3400 50  0001 C CNN
 F 3 "" H 5600 3400 50  0001 C CNN
+F 4 "P150KDBCT-ND" V 5600 3400 60  0001 C CNN "Digikey"
 	1    5600 3400
 	0    1    1    0
@@
 F 2 "footprints:CR43NP-4R7MC" H 7300 3100 50  0001 C CNN
 F 3 "" H 7300 3100 50  0001 C CNN
+F 4 "308-1527-1-ND" V 7300 3100 60  0001 C CNN "Digikey"
 	1    7300 3100
 	0    1    1    0
@@
 F 2 "footprints:R_0603" V 5830 3150 50  0001 C CNN
 F 3 "" H 5900 3150 50  0001 C CNN
+F 4 "A119962CT-ND" V 5900 3150 60  0001 C CNN "Digikey"
 	1    5900 3150
 	1    0    0    -1
@@
 F 2 "footprints:CP_Elec_4x4.5" H 7588 3150 50  0001 C CNN
 F 3 "" H 7550 3300 50  0001 C CNN
+F 4 "PCE3878CT-ND" H 7550 3300 60  0001 C CNN "Digikey"
 	1    7550 3300
 	1    0    0    -1
@@
 P 7800 3300
 F 0 "C33" H 7700 3200 50  0000 L CNN
-F 1 "103" H 7650 3400 50  0000 L CNN
+F 1 "10nF" H 7650 3400 50  0000 L CNN
 F 2 "footprints:C_0603" H 7838 3150 50  0001 C CNN
 F 3 "" H 7800 3300 50  0001 C CNN
+F 4 "478-1227-1-ND" H 7800 3300 60  0001 C CNN "Digikey"
 	1    7800 3300
 	-1   0    0    1
@@
 F 2 "footprints:L_0603" H 8150 3100 50  0001 C CNN
 F 3 "" H 8150 3100 50  0001 C CNN
+F 4 "490-14398-2-ND" V 8150 3100 60  0001 C CNN "Digikey"
 	1    8150 3100
 	0    1    1    0
@@
 F 2 "footprints:L_0603" H 10500 1000 50  0001 C CNN
 F 3 "" H 10500 1000 50  0001 C CNN
+F 4 "490-14398-2-ND" V 10500 1000 60  0001 C CNN "Digikey"
 	1    10500 1000
 	0    1    1    0
@@
 F 2 "footprints:L_0603" H 10500 1150 50  0001 C CNN
 F 3 "" H 10500 1150 50  0001 C CNN
+F 4 "490-14398-2-ND" V 10500 1150 60  0001 C CNN "Digikey"
 	1    10500 1150
 	0    1    1    0
@@
 F 2 "footprints:L_0603" H 10500 1350 50  0001 C CNN
 F 3 "" H 10500 1350 50  0001 C CNN
+F 4 "490-14398-2-ND" V 10500 1350 60  0001 C CNN "Digikey"
 	1    10500 1350
 	0    1    1    0
@@
 F 2 "footprints:R_0603" V 9680 1600 50  0001 C CNN
 F 3 "" H 9750 1600 50  0001 C CNN
+F 4 "A103049TR-ND" V 9750 1600 60  0001 C CNN "Digikey"
 	1    9750 1600
 	1    0    0    -1
@@
 F 2 "footprints:R_0603" V 9880 1600 50  0001 C CNN
 F 3 "" H 9950 1600 50  0001 C CNN
+F 4 "A103049TR-ND" V 9950 1600 60  0001 C CNN "Digikey"
 	1    9950 1600
 	1    0    0    -1
@@
 P 9750 1950
 F 0 "C39" V 9800 2000 50  0000 L CNN
-F 1 "473" V 9700 2000 50  0000 L CNN
+F 1 "47nF" V 9700 2000 50  0000 L CNN
 F 2 "footprints:C_0603" H 9788 1800 50  0001 C CNN
 F 3 "" H 9750 1950 50  0001 C CNN
+F 4 "399-9096-1-ND" V 9750 1950 60  0001 C CNN "Digikey"
 	1    9750 1950
 	-1   0    0    1
@@
 P 9950 1950
 F 0 "C40" V 10000 2000 50  0000 L CNN
-F 1 "473" V 9900 2000 50  0000 L CNN
+F 1 "47nF" V 9900 2000 50  0000 L CNN
 F 2 "footprints:C_0603" H 9988 1800 50  0001 C CNN
 F 3 "" H 9950 1950 50  0001 C CNN
+F 4 "399-9096-1-ND" V 9950 1950 60  0001 C CNN "Digikey"
 	1    9950 1950
 	-1   0    0    1
@@
 F 2 "footprints:L_0603" H 10550 2200 50  0001 C CNN
 F 3 "" H 10550 2200 50  0001 C CNN
+F 4 "490-14398-2-ND" V 10550 2200 60  0001 C CNN "Digikey"
 	1    10550 2200
 	0    1    1    0
@@
 F 2 "footprints:L_0603" H 10550 2350 50  0001 C CNN
 F 3 "" H 10550 2350 50  0001 C CNN
+F 4 "490-14398-2-ND" V 10550 2350 60  0001 C CNN "Digikey"
 	1    10550 2350
 	0    1    1    0
@@
 F 2 "footprints:C_0603" H 12888 1400 50  0001 C CNN
 F 3 "" H 12850 1550 50  0001 C CNN
+F 4 "399-1095-1-ND" V 12850 1550 60  0001 C CNN "Digikey"
 	1    12850 1550
 	0    -1   -1   0
@@
 F 2 "footprints:R_0603" V 12230 2250 50  0001 C CNN
 F 3 "" H 12300 2250 50  0001 C CNN
+F 4 "311-10KDCT-ND" V 12300 2250 60  0001 C CNN "Digikey"
 	1    12300 2250
 	1    0    0    -1
@@
 F 2 "footprints:R_0603" V 12630 2250 50  0001 C CNN
 F 3 "" H 12700 2250 50  0001 C CNN
+F 4 "311-10KDCT-ND" V 12700 2250 60  0001 C CNN "Digikey"
 	1    12700 2250
 	1    0    0    -1
@@
 F 2 "footprints:C_0603" H 12538 2800 50  0001 C CNN
 F 3 "" H 12500 2950 50  0001 C CNN
+F 4 "399-1095-1-ND" H 12500 2950 60  0001 C CNN "Digikey"
 	1    12500 2950
 	1    0    0    -1
@@
 F 2 "footprints:C_0603" H 13288 4300 50  0001 C CNN
 F 3 "" H 13250 4450 50  0001 C CNN
+F 4 "399-1095-1-ND" H 13250 4450 60  0001 C CNN "Digikey"
 	1    13250 4450
 	1    0    0    -1
@@
 F 2 "footprints:R_0603" V 13780 1850 50  0001 C CNN
 F 3 "" H 13850 1850 50  0001 C CNN
+F 4 "MCT0603-33.0-CFCT-ND" V 13850 1850 60  0001 C CNN "Digikey"
 	1    13850 1850
 	0    1    1    0
@@
 F 2 "footprints:R_0603" V 13780 1950 50  0001 C CNN
 F 3 "" H 13850 1950 50  0001 C CNN
+F 4 "MCT0603-33.0-CFCT-ND" V 13850 1950 60  0001 C CNN "Digikey"
 	1    13850 1950
 	0    1    1    0
@@
 F 2 "footprints:R_0603" V 13780 2050 50  0001 C CNN
 F 3 "" H 13850 2050 50  0001 C CNN
+F 4 "MCT0603-33.0-CFCT-ND" V 13850 2050 60  0001 C CNN "Digikey"
 	1    13850 2050
 	0    1    1    0
@@
 F 2 "footprints:R_0603" V 13780 2150 50  0001 C CNN
 F 3 "" H 13850 2150 50  0001 C CNN
+F 4 "MCT0603-33.0-CFCT-ND" V 13850 2150 60  0001 C CNN "Digikey"
 	1    13850 2150
 	0    1    1    0
